Commit message: E. Joints abs & rel coords done

File: body.urdf (robot description, URDF)
Before this commit: robot robot, 2 links, 1 joints
Links:
- removed link leg
- removed link torso
- added link link0, mass 1; collision box size=1 1 1; visual box size=1 1 1
- added link link1, mass 1; collision box size=1 1 1; visual box size=1 1 1
- added link link2, mass 1; collision box size=1 1 1; visual box size=1 1 1
- added link link3, mass 1; collision box size=1 1 1; visual box size=1 1 1
- added link link4, mass 1; collision box size=1 1 1; visual box size=1 1 1
- added link link5, mass 1; collision box size=1 1 1; visual box size=1 1 1
- added link link6, mass 1; collision box size=1 1 1; visual box size=1 1 1
Joints:
- removed joint Torso_Leg
- added joint link0_link1: type revolute, parent link0, child link1, origin xyz=0 0 1 rpy=0 0 0, axis 0 1 0, limit lower=-3.14159 upper=3.14159 effort=0.0 velocity=0.0
- added joint link1_link2: type revolute, parent link1, child link2, origin xyz=0 0 1 rpy=0 0 0, axis 0 1 0, limit lower=-3.14159 upper=3.14159 effort=0.0 velocity=0.0
- added joint link2_link3: type revolute, parent link2, child link3, origin xyz=0.5 0 0.5 rpy=0 0 0, axis 0 1 0, limit lower=-3.14159 upper=3.14159 effort=0.0 velocity=0.0
- added joint link3_link4: type revolute, parent link3, child link4, origin xyz=1 0 0 rpy=0 0 0, axis 0 1 0, limit lower=-3.14159 upper=3.14159 effort=0.0 velocity=0.0
- added joint link4_link5: type revolute, parent link4, child link5, origin xyz=0.5 0 -0.5 rpy=0 0 0, axis 0 1 0, limit lower=-3.14159 upper=3.14159 effort=0.0 velocity=0.0
- added joint link5_link6: type revolute, parent link5, child link6, origin xyz=0 0 -1 rpy=0 0 0, axis 0 1 0, limit lower=-3.14159 upper=3.14159 effort=0.0 velocity=0.0

Commit message: E. joints done

File: body.urdf (robot description, URDF)
Before this commit: robot robot, 7 links, 6 joints
Links:
- removed link link0
- removed link link1
- removed link link2
- removed link link3
- removed link link4
- removed link link5
- removed link link6
- added link Backleg, mass 1; collision box size=1 1 1; visual box size=1 1 1
- added link Frontleg, mass 1; collision box size=1 1 1; visual box size=1 1 1
- added link Torso, mass 1; collision box size=1 1 1; visual box size=1 1 1
Joints:
- removed joint link0_link1
- removed joint link1_link2
- removed joint link2_link3
- removed joint link3_link4
- removed joint link4_link5
- removed joint link5_link6
- added joint Torso_Backleg: type revolute, parent Torso, child Backleg, origin xyz=1 0 1 rpy=0 0 0, axis 0 1 0, limit lower=-3.14159 upper=3.14159 effort=0.0 velocity=0.0
- added joint Torso_Frontleg: type revolute, parent Torso, child Frontleg, origin xyz=2 0 1 rpy=0 0 0, axis 0 1 0, limit lower=-3.14159 upper=3.14159 effort=0.0 velocity=0.0

Commit message: N. quadruped done

File: body.urdf (robot description, URDF)
Before this commit: robot robot, 3 links, 2 joints
Links:
- added link BackLowerleg, mass 1; collision box size=0.2 0.2 1; visual box size=0.2 0.2 1
- added link FrontLowerleg, mass 1; collision box size=0.2 0.2 1; visual box size=0.2 0.2 1
- added link LeftLowerleg, mass 1; collision box size=0.2 0.2 1; visual box size=0.2 0.2 1
- added link Leftleg, mass 1; collision box size=1 0.2 0.2; visual box size=1 0.2 0.2
- added link RightLowerleg, mass 1; collision box size=0.2 0.2 1; visual box size=0.2 0.2 1
- added link Rightleg, mass 1; collision box size=1 0.2 0.2; visual box size=1 0.2 0.2
- link Backleg: geometry collision box size=0.2 1 0.2; visual box size=0.2 1 0.2
- link Frontleg: geometry collision box size=0.2 1 0.2; visual box size=0.2 1 0.2
Joints:
- added joint Backleg_BackLowerleg: type revolute, parent Backleg, child BackLowerleg, origin xyz=0 -1 0 rpy=0 0 0, axis 1 0 0, limit lower=-3.14159 upper=3.14159 effort=0.0 velocity=0.0
- added joint Frontleg_FrontLowerleg: type revolute, parent Frontleg, child FrontLowerleg, origin xyz=0 1 0 rpy=0 0 0, axis 1 0 0, limit lower=-3.14159 upper=3.14159 effort=0.0 velocity=0.0
- added joint Leftleg_LeftLowerleg: type revolute, parent Leftleg, child LeftLowerleg, origin xyz=-1 0 0 rpy=0 0 0, axis 0 1 0, limit lower=-3.14159 upper=3.14159 effort=0.0 velocity=0.0
- added joint Rightleg_RightLowerleg: type revolute, parent Rightleg, child RightLowerleg, origin xyz=1 0 0 rpy=0 0 0, axis 0 1 0, limit lower=-3.14159 upper=3.14159 effort=0.0 velocity=0.0
- added joint Torso_Leftleg: type revolute, parent Torso, child Leftleg, origin xyz=-0.5 0 1 rpy=0 0 0, axis 0 1 0, limit lower=-3.14159 upper=3.14159 effort=0.0 velocity=0.0
- added joint Torso_Rightleg: type revolute, parent Torso, child Rightleg, origin xyz=0.5 0 1 rpy=0 0 0, axis 0 1 0, limit lower=-3.14159 upper=3.14159 effort=0.0 velocity=0.0
- joint Torso_Backleg: axis 0 1 0 -> 1 0 0; origin xyz=1 0 1 rpy=0 0 0 -> xyz=0 -0.5 1 rpy=0 0 0
- joint Torso_Frontleg: axis 0 1 0 -> 1 0 0; origin xyz=2 0 1 rpy=0 0 0 -> xyz=0 0.5 1 rpy=0 0 0

Commit message: assgmt5 jumper done

File: body.urdf (robot description, URDF)
Before this commit: robot robot, 9 links, 8 joints
Links:
- added link Backarm, mass 1; collision box size=1.5 0.2 0.2; visual box size=1.5 0.2 0.2
- added link Frontarm, mass 1; collision box size=1.5 0.2 0.2; visual box size=1.5 0.2 0.2
- added link Leftarm, mass 1; collision box size=0.2 1.5 0.2; visual box size=0.2 1.5 0.2
- added link Rightarm, mass 1; collision box size=0.2 1.5 0.2; visual box size=0.2 1.5 0.2
- link BackLowerleg: geometry collision box size=0.5 0.25 0.25; visual box size=0.5 0.25 0.25
- link Backleg: geometry collision box size=0.2 0.2 0.5; visual box size=0.2 0.2 0.5
- link FrontLowerleg: geometry collision box size=0.5 0.25 0.25; visual box size=0.5 0.25 0.25
- link Frontleg: geometry collision box size=0.2 0.2 0.5; visual box size=0.2 0.2 0.5
- link LeftLowerleg: geometry collision box size=0.5 0.25 0.25; visual box size=0.5 0.25 0.25
- link Leftleg: geometry collision box size=0.2 0.2 0.5; visual box size=0.2 0.2 0.5
- link RightLowerleg: geometry collision box size=0.5 0.25 0.25; visual box size=0.5 0.25 0.25
- link Rightleg: geometry collision box size=0.2 0.2 0.5; visual box size=0.2 0.2 0.5
Joints:
- added joint Torso_Backarm: type revolute, parent Torso, child Backarm, origin xyz=0.5 0 2 rpy=0 0 0, axis 0 1 0, limit lower=-3.14159 upper=3.14159 effort=0.0 velocity=0.0
- added joint Torso_Frontarm: type revolute, parent Torso, child Frontarm, origin xyz=-0.5 0 2 rpy=0 0 0, axis 0 1 0, limit lower=-3.14159 upper=3.14159 effort=0.0 velocity=0.0
- added joint Torso_Leftarm: type revolute, parent Torso, child Leftarm, origin xyz=0 -0.5 2 rpy=0 0 0, axis 1 0 0, limit lower=-3.14159 upper=3.14159 effort=0.0 velocity=0.0
- added joint Torso_Rightarm: type revolute, parent Torso, child Rightarm, origin xyz=0 0.5 2 rpy=0 0 0, axis 1 0 0, limit lower=-3.14159 upper=3.14159 effort=0.0 velocity=0.0
- joint Backleg_BackLowerleg: axis 1 0 0 -> 0 1 0; origin xyz=0 -1 0 rpy=0 0 0 -> xyz=0 0 -0.5 rpy=0 0 0
- joint Frontleg_FrontLowerleg: axis 1 0 0 -> 0 1 0; origin xyz=0 1 0 rpy=0 0 0 -> xyz=0 0 -0.5 rpy=0 0 0
- joint Leftleg_LeftLowerleg: origin xyz=-1 0 0 rpy=0 0 0 -> xyz=0 0 -0.5 rpy=0 0 0
- joint Rightleg_RightLowerleg: origin xyz=1 0 0 rpy=0 0 0 -> xyz=0 0 -0.5 rpy=0 0 0
- joint Torso_Backleg: axis 1 0 0 -> 0 1 0; origin xyz=0 -0.5 1 rpy=0 0 0 -> xyz=0.25 0.25 1.5 rpy=0 0 0
- joint Torso_Frontleg: axis 1 0 0 -> 0 1 0; origin xyz=0 0.5 1 rpy=0 0 0 -> xyz=-0.25 0.25 1.5 rpy=0 0 0
- joint Torso_Leftleg: origin xyz=-0.5 0 1 rpy=0 0 0 -> xyz=-0.25 -0.25 1.5 rpy=0 0 0
- joint Torso_Rightleg: origin xyz=0.5 0 1 rpy=0 0 0 -> xyz=0.25 -0.25 1.5 rpy=0 0 0

Commit message: generate random shapes and sensors, need to check poitions and change color

File: body.urdf (robot description, URDF)
Before this commit: robot robot, 13 links, 12 joints
Links:
- removed link BackLowerleg
- removed link Backarm
- removed link Backleg
- removed link FrontLowerleg
- removed link Frontarm
- removed link Frontleg
- removed link LeftLowerleg
- removed link Leftarm
- removed link Leftleg
- removed link RightLowerleg
- removed link Rightarm
- removed link Rightleg
- removed link Torso
- added link Head, mass 1; collision sphere radius=1; visual sphere radius=1
- added link link0, mass 1; collision sphere radius=1.9069022880121609; visual sphere radius=1.9069022880121609
Joints:
- removed joint Backleg_BackLowerleg
- removed joint Frontleg_FrontLowerleg
- removed joint Leftleg_LeftLowerleg
- removed joint Rightleg_RightLowerleg
- removed joint Torso_Backarm
- removed joint Torso_Backleg
- removed joint Torso_Frontarm
- removed joint Torso_Frontleg
- removed joint Torso_Leftarm
- removed joint Torso_Leftleg
- removed joint Torso_Rightarm
- removed joint Torso_Rightleg
- added joint Head_link0: type revolute, parent Head, child link0, origin xyz=1 0 0 rpy=0 0 0, axis 0 1 0, limit lower=-3.14159 upper=3.14159 effort=0.0 velocity=0.0

Commit message: figure out colors and rest of pos

File: body.urdf (robot description, URDF)
Before this commit: robot robot, 2 links, 1 joints
Links:
- added link link1, mass 1; collision sphere radius=1.9874150029985824; visual sphere radius=1.9874150029985824
- added link link2, mass 1; collision cylinder length=1.993085282189517 radius=1.0686548516861993; visual cylinder length=1.993085282189517 radius=1.0686548516861993
- added link link3, mass 1; collision box size=1.8627014607073953 1.3741938592792844 1.3020659835101362; visual box size=1.8627014607073953 1.3741938592792844 1.3020659835101362
- link Head: geometry collision box size=4 4 4; visual box size=4 4 4
- link link0: geometry collision box size=1.941281124102094 1.066471943189216 1.458515503071564; visual box size=1.941281124102094 1.066471943189216 1.458515503071564
Joints:
- added joint link0_link1: type revolute, parent link0, child link1, origin xyz=-1.941281124102094 0 0 rpy=0 0 0, axis 0 0 1, limit lower=-3.14159 upper=3.14159 effort=0.0 velocity=0.0
- added joint link1_link2: type revolute, parent link1, child link2, origin xyz=-1.9874150029985824 0 0 rpy=0 0 0, axis 0 0 1, limit lower=-3.14159 upper=3.14159 effort=0.0 velocity=0.0
- added joint link2_link3: type revolute, parent link2, child link3, origin xyz=-1.993085282189517 0 0 rpy=0 0 0, axis 0 0 1, limit lower=-3.14159 upper=3.14159 effort=0.0 velocity=0.0
- joint Head_link0: axis 0 1 0 -> 0 0 1; origin xyz=1 0 0 rpy=0 0 0 -> xyz=-2 0 1 rpy=0 0 0

Commit message: assgmt6 done

File: body.urdf (robot description, URDF)
Before this commit: robot robot, 5 links, 4 joints
Links:
- removed link Head
- added link link4, mass 1; collision cylinder length=1.3570683533476737 radius=0.6785341766738369; visual cylinder length=1.3570683533476737 radius=0.6785341766738369
- link link0: geometry collision sphere radius=0.5; visual sphere radius=0.5
- link link1: geometry collision box size=1.687729272277555 0.5238130031864603 0.9417455161882976; visual box size=1.687729272277555 0.5238130031864603 0.9417455161882976
- link link2: geometry collision sphere radius=0.8464222377057053; visual sphere radius=0.8464222377057053
- link link3: geometry collision sphere radius=0.5398728726720308; visual sphere radius=0.5398728726720308
Joints:
- removed joint Head_link0
- added joint link3_link4: type revolute, parent link3, child link4, origin xyz=-1.0797457453440615 0 0 rpy=0 0 0, axis 0 0 1, limit lower=-3.14159 upper=3.14159 effort=0.0 velocity=0.0
- joint link0_link1: origin xyz=-1.941281124102094 0 0 rpy=0 0 0 -> xyz=-0.5 0 1 rpy=0 0 0
- joint link1_link2: origin xyz=-1.9874150029985824 0 0 rpy=0 0 0 -> xyz=-1.687729272277555 0 0 rpy=0 0 0
- joint link2_link3: origin xyz=-1.993085282189517 0 0 rpy=0 0 0 -> xyz=-1.6928444754114107 0 0 rpy=0 0 0

Commit message: assgmt7 so far. may remove dir

File: body.urdf (robot description, URDF)
Before this commit: robot robot, 5 links, 4 joints
Links:
- removed link link2
- removed link link3
- removed link link4
- link link0: geometry collision box size=1 1 1; visual box size=1 1 1
- link link1: geometry collision box size=0.6677380291036654 0.9270864501590491 0.7635717993594329; visual box size=0.6677380291036654 0.9270864501590491 0.7635717993594329
Joints:
- removed joint link1_link2
- removed joint link2_link3
- removed joint link3_link4
- joint link0_link1: axis 0 0 1 -> 0 1 0; origin xyz=-0.5 0 1 rpy=0 0 0 -> xyz=0 -0.5 3 rpy=0 0 0

Commit message: assgmt7 done

File: body.urdf (robot description, URDF)
Before this commit: robot robot, 2 links, 1 joints
Links:
- added link link2, mass 1; collision box size=0.9885591297559984 0.9885591297559984 0.9885591297559984; visual box size=0.9885591297559984 0.9885591297559984 0.9885591297559984
- added link link3, mass 1; collision box size=0.5418345991518301 0.5418345991518301 0.5418345991518301; visual box size=0.5418345991518301 0.5418345991518301 0.5418345991518301
- added link link4, mass 1; collision cylinder length=0.6958351409395724 radius=0.3479175704697862; visual cylinder length=0.6958351409395724 radius=0.3479175704697862
- link link1: geometry collision cylinder length=0.7691604926919615 radius=0.38458024634598076; visual cylinder length=0.7691604926919615 radius=0.38458024634598076
Joints:
- added joint link1_link2: type revolute, parent link1, child link2, origin xyz=-0.38458024634598076 -0.38458024634598076 0 rpy=0 0 0, axis 1 0 0, limit lower=-3.14159 upper=3.14159 effort=0.0 velocity=0.0
- added joint link2_link3: type revolute, parent link2, child link3, origin xyz=-0.4942795648779992 0 -0.4942795648779992 rpy=0 0 0, axis 0 0 1, limit lower=-3.14159 upper=3.14159 effort=0.0 velocity=0.0
- added joint link3_link4: type revolute, parent link3, child link4, origin xyz=-0.27091729957591504 0 -0.27091729957591504 rpy=0 0 0, axis 1 0 0, limit lower=-3.14159 upper=3.14159 effort=0.0 velocity=0.0

Commit message: with shapes

File: body.urdf (robot description, URDF)
Before this commit: robot robot, 5 links, 4 joints
Links:
- link link0: geometry collision cylinder length=1 radius=0.5; visual cylinder length=1 radius=0.5
- link link1: geometry collision sphere radius=0.35341592532774846; visual sphere radius=0.35341592532774846
- link link2: geometry collision sphere radius=0.3844380958842861; visual sphere radius=0.3844380958842861
- link link3: geometry collision box size=0.5401558606380494 0.5401558606380494 0.05397200811037284; visual box size=0.5401558606380494 0.5401558606380494 0.05397200811037284
- link link4: geometry collision box size=0.8148305468189769 0.8148305468189769 0.8148305468189769; visual box size=0.8148305468189769 0.8148305468189769 0.8148305468189769
Joints:
- joint link0_link1: origin xyz=0 -0.5 3 rpy=0 0 0 -> xyz=0 -0.5 5 rpy=0 0 0
- joint link1_link2: axis 1 0 0 -> 0 0 1; origin xyz=-0.38458024634598076 -0.38458024634598076 0 rpy=0 0 0 -> xyz=0 0 4.5 rpy=0 0 0
- joint link2_link3: axis 0 0 1 -> 1 0 0; origin xyz=-0.4942795648779992 0 -0.4942795648779992 rpy=0 0 0 -> xyz=-0.3844380958842861 -0.3844380958842861 0 rpy=0 0 0
- joint link3_link4: axis 1 0 0 -> 0 1 0; origin xyz=-0.27091729957591504 0 -0.27091729957591504 rpy=0 0 0 -> xyz=0 -0.2700779303190247 -0.02698600405518642 rpy=0 0 0

Commit message: assgmt 8 done

File: body.urdf (robot description, URDF)
Before this commit: robot robot, 5 links, 4 joints
Links:
- link link1: geometry collision box size=0.5685382151693721 0.5685382151693721 0.5685382151693721; visual box size=0.5685382151693721 0.5685382151693721 0.5685382151693721
- link link2: geometry collision box size=0.7349986211288271 0.7349986211288271 0.7349986211288271; visual box size=0.7349986211288271 0.7349986211288271 0.7349986211288271
- link link3: geometry collision sphere radius=0.4012288093919565; visual sphere radius=0.4012288093919565
- link link4: geometry collision cylinder length=0.6361402586116705 radius=0.3180701293058352; visual cylinder length=0.6361402586116705 radius=0.3180701293058352
Joints:
- joint link0_link1: axis 0 1 0 -> 1 0 0; origin xyz=0 -0.5 5 rpy=0 0 0 -> xyz=-0.5 0 5 rpy=0 0 0
- joint link1_link2: axis 0 0 1 -> 1 0 0; origin xyz=0 0 4.5 rpy=0 0 0 -> xyz=-0.5685382151693721 0 0 rpy=0 0 0
- joint link2_link3: axis 1 0 0 -> 0 1 0; origin xyz=-0.3844380958842861 -0.3844380958842861 0 rpy=0 0 0 -> xyz=-0.36749931056441354 -0.36749931056441354 0 rpy=0 0 0
- joint link3_link4: origin xyz=0 -0.2700779303190247 -0.02698600405518642 rpy=0 0 0 -> xyz=-0.4954732102513761 -0.4012288093919565 0 rpy=0 0 0

Commit message: refactored, added type argument

File: body.urdf (robot description, URDF)
Before this commit: robot robot, 5 links, 4 joints
Links:
- link link0: geometry collision box size=1 1 1; visual box size=1 1 1
- link link1: geometry collision box size=0.7395317052219721 0.5100799975631303 0.8231839575782907; visual box size=0.7395317052219721 0.5100799975631303 0.8231839575782907
- link link2: geometry collision box size=0.5072467653992154 0.7458173777397457 0.7810538484814917; visual box size=0.5072467653992154 0.7458173777397457 0.7810538484814917
- link link3: geometry collision box size=0.6818582550293186 0.9290021001292696 0.5016080650883225; visual box size=0.6818582550293186 0.9290021001292696 0.5016080650883225
- link link4: geometry collision box size=0.9552757611638436 0.5200623126070111 0.9756626471966932; visual box size=0.9552757611638436 0.5200623126070111 0.9756626471966932
Joints:
- joint link0_link1: origin xyz=-0.5 0 5 rpy=0 0 0 -> xyz=0 0 5.5 rpy=0 0 0
- joint link1_link2: origin xyz=-0.5685382151693721 0 0 rpy=0 0 0 -> xyz=0 0.25503999878156514 0.41159197878914533 rpy=0 0 0
- joint link2_link3: axis 0 1 0 -> 1 0 0; origin xyz=-0.36749931056441354 -0.36749931056441354 0 rpy=0 0 0 -> xyz=0.2536233826996077 0.37290868886987283 0 rpy=0 0 0
- joint link3_link4: axis 0 1 0 -> 1 0 0; origin xyz=-0.4954732102513761 -0.4012288093919565 0 rpy=0 0 0 -> xyz=0.3409291275146593 0.4645010500646348 0 rpy=0 0 0
