Commit message: final

File: save/0body.urdf (robot description, URDF)
Before this commit: robot robot, 4 links, 3 joints
Links:
- added link link4, mass 1; collision box size=0.8248803024737357 0.3006391952727901 0.41575918239049187; visual box size=0.8248803024737357 0.3006391952727901 0.41575918239049187
- added link link5, mass 1; collision box size=0.6440351137341451 0.6458066949495007 0.797402078779464; visual box size=0.6440351137341451 0.6458066949495007 0.797402078779464
- added link link6, mass 1; collision box size=0.21076969630471043 0.3727468062012249 0.5082914179940438; visual box size=0.21076969630471043 0.3727468062012249 0.5082914179940438
- added link link7, mass 1; collision box size=0.5619008774083376 0.8430422025160806 0.3853927416352213; visual box size=0.5619008774083376 0.8430422025160806 0.3853927416352213
- added link link8, mass 1; collision box size=0.24614070536855506 0.8968343971369444 0.37920432020991823; visual box size=0.24614070536855506 0.8968343971369444 0.37920432020991823
- link link0: geometry collision box size=0.6930622950576663 0.6692507471486218 0.5667899052389529; visual box size=0.6930622950576663 0.6692507471486218 0.5667899052389529
- link link1: geometry collision box size=0.3718531290576076 0.3703445166878872 0.795443292181671; visual box size=0.3718531290576076 0.3703445166878872 0.795443292181671
- link link2: geometry collision box size=0.2755903137222566 0.6492327220839093 0.5911744749561743; visual box size=0.2755903137222566 0.6492327220839093 0.5911744749561743
- link link3: geometry collision box size=0.8385876845184308 0.6799383925200941 0.4438362674922669; visual box size=0.8385876845184308 0.6799383925200941 0.4438362674922669
Joints:
- added joint link3_link4: type revolute, parent link3, child link4, origin xyz=0.4192938422592154 0 0.22191813374613345 rpy=0 0 0, axis 1 0 0, limit lower=-3.14159 upper=3.14159 effort=0.0 velocity=0.0
- added joint link4_link5: type revolute, parent link4, child link5, origin xyz=0 0 0.41575918239049187 rpy=0 0 0, axis 1 0 0, limit lower=-3.14159 upper=3.14159 effort=0.0 velocity=0.0
- added joint link5_link6: type revolute, parent link5, child link6, origin xyz=0 0 0.797402078779464 rpy=0 0 0, axis 1 0 0, limit lower=-3.14159 upper=3.14159 effort=0.0 velocity=0.0
- added joint link6_link7: type revolute, parent link6, child link7, origin xyz=0 0.18637340310061246 0.2541457089970219 rpy=0 0 0, axis 1 0 0, limit lower=-3.14159 upper=3.14159 effort=0.0 velocity=0.0
- added joint link7_link8: type revolute, parent link7, child link8, origin xyz=0 0.4215211012580403 0.19269637081761065 rpy=0 0 0, axis 1 0 0, limit lower=-3.14159 upper=3.14159 effort=0.0 velocity=0.0
- joint link0_link1: origin xyz=0.25 0 5 rpy=0 0 0 -> xyz=0 0.3346253735743109 5 rpy=0 0 0
- joint link1_link2: origin xyz=0.29117879501151855 0.12328650741576519 0 rpy=0 0 0 -> xyz=0 0.1851722583439436 0.3977216460908355 rpy=0 0 0
- joint link2_link3: origin xyz=0.10721772569730931 0.20950158310254668 0 rpy=0 0 0 -> xyz=0.1377951568611283 0 0.29558723747808713 rpy=0 0 0

File: save/1body.urdf (robot description, URDF)
Before this commit: robot robot, 4 links, 3 joints
Links:
- added link link4, mass 1; collision box size=0.24859281761157048 0.5510039311174055 0.42758240756239935; visual box size=0.24859281761157048 0.5510039311174055 0.42758240756239935
- added link link5, mass 1; collision box size=0.49636712382087533 0.6991616180567579 0.503647667964993; visual box size=0.49636712382087533 0.6991616180567579 0.503647667964993
- link link1: geometry collision box size=0.5009024926493721 0.9679977211647273 0.9073001502543006; visual box size=0.5009024926493721 0.9679977211647273 0.9073001502543006
- link link2: geometry collision box size=0.24640166199832142 0.822493974209175 0.7669345233045386; visual box size=0.24640166199832142 0.822493974209175 0.7669345233045386
- link link3: geometry collision box size=0.855637493647492 0.5151121967256231 0.2705906376096356; visual box size=0.855637493647492 0.5151121967256231 0.2705906376096356
Joints:
- added joint link3_link4: type revolute, parent link3, child link4, origin xyz=0.427818746823746 0 0.1352953188048178 rpy=0 0 0, axis 0 0 1, limit lower=-3.14159 upper=3.14159 effort=0.0 velocity=0.0
- added joint link4_link5: type revolute, parent link4, child link5, origin xyz=0 0 0.42758240756239935 rpy=0 0 0, axis 0 0 1, limit lower=-3.14159 upper=3.14159 effort=0.0 velocity=0.0
- joint link0_link1: axis 0 1 0 -> 0 0 1; origin xyz=0 0 5.25 rpy=0 0 0 -> xyz=0 0.25 5 rpy=0 0 0
- joint link1_link2: axis 0 1 0 -> 0 0 1; origin xyz=0 0 0.28049019936898917 rpy=0 0 0 -> xyz=0.25045124632468607 0.48399886058236363 0 rpy=0 0 0
- joint link2_link3: axis 0 1 0 -> 0 0 1; origin xyz=0.37376036201938767 0 0.4679139383223354 rpy=0 0 0 -> xyz=0.24640166199832142 0 0 rpy=0 0 0

File: save/2body.urdf (robot description, URDF)
Before this commit: robot robot, 4 links, 3 joints
Links:
- link link1: geometry collision box size=0.8720421348018628 0.5431086801714589 0.28049019936898917; visual box size=0.8720421348018628 0.5431086801714589 0.28049019936898917
- link link2: geometry collision box size=0.7475207240387753 0.5433567844305411 0.9358278766446708; visual box size=0.7475207240387753 0.5433567844305411 0.9358278766446708
- link link3: geometry collision box size=0.5473978557829923 0.4897504849884926 0.7978930276887026; visual box size=0.5473978557829923 0.4897504849884926 0.7978930276887026
Joints:
- joint link0_link1: axis 1 0 0 -> 0 1 0; origin xyz=0 0.25 5 rpy=0 0 0 -> xyz=0 0 5.25 rpy=0 0 0
- joint link1_link2: axis 1 0 0 -> 0 1 0; origin xyz=0.29688399905636 0.2821946827708924 0 rpy=0 0 0 -> xyz=0 0 0.28049019936898917 rpy=0 0 0
- joint link2_link3: axis 1 0 0 -> 0 1 0; origin xyz=0.8537089899008325 0 0 rpy=0 0 0 -> xyz=0.37376036201938767 0 0.4679139383223354 rpy=0 0 0

File: save/3body.urdf (robot description, URDF)
Before this commit: robot robot, 4 links, 3 joints
Links:
- added link link4, mass 1; collision box size=0.34827928290455235 0.9312777014039482 0.4838147804160149; visual box size=0.34827928290455235 0.9312777014039482 0.4838147804160149
- added link link5, mass 1; collision box size=0.32693649511917144 0.28928596076655844 0.9364238750962248; visual box size=0.32693649511917144 0.28928596076655844 0.9364238750962248
- link link1: geometry collision box size=0.35016657174002735 0.3171655306013579 0.7929080199525589; visual box size=0.35016657174002735 0.3171655306013579 0.7929080199525589
- link link2: geometry collision box size=0.7104967845277153 0.48653808148604993 0.6880599860451834; visual box size=0.7104967845277153 0.48653808148604993 0.6880599860451834
- link link3: geometry collision box size=0.5375914729147773 0.21971262009818898 0.3346389493270204; visual box size=0.5375914729147773 0.21971262009818898 0.3346389493270204
Joints:
- added joint link3_link4: type revolute, parent link3, child link4, origin xyz=0.26879573645738863 0.10985631004909449 0 rpy=0 0 0, axis 0 1 0, limit lower=-3.14159 upper=3.14159 effort=0.0 velocity=0.0
- added joint link4_link5: type revolute, parent link4, child link5, origin xyz=0 0.4656388507019741 0.24190739020800744 rpy=0 0 0, axis 0 1 0, limit lower=-3.14159 upper=3.14159 effort=0.0 velocity=0.0
- joint link1_link2: origin xyz=0.23070226369644165 0 0.13726656219869324 rpy=0 0 0 -> xyz=0 0 0.7929080199525589 rpy=0 0 0
- joint link2_link3: origin xyz=0.4643223742066076 0 0.12369040386078184 rpy=0 0 0 -> xyz=0.3552483922638576 0 0.3440299930225917 rpy=0 0 0

File: save/4body.urdf (robot description, URDF)
Before this commit: robot robot, 4 links, 3 joints
Links:
- link link1: geometry collision box size=0.4614045273928833 0.20266338237334525 0.2745331243973865; visual box size=0.4614045273928833 0.20266338237334525 0.2745331243973865
- link link2: geometry collision box size=0.9286447484132152 0.5945031053927179 0.24738080772156368; visual box size=0.9286447484132152 0.5945031053927179 0.24738080772156368
- link link3: geometry collision box size=0.5381354021658709 0.34318753609538477 0.47926415177749215; visual box size=0.5381354021658709 0.34318753609538477 0.47926415177749215
Joints:
- joint link0_link1: axis 0 0 1 -> 0 1 0
- joint link1_link2: axis 0 0 1 -> 0 1 0; origin xyz=0 0 0.3156967477942252 rpy=0 0 0 -> xyz=0.23070226369644165 0 0.13726656219869324 rpy=0 0 0
- joint link2_link3: axis 0 0 1 -> 0 1 0; origin xyz=0.1415789467550313 0 0.18682523893142391 rpy=0 0 0 -> xyz=0.4643223742066076 0 0.12369040386078184 rpy=0 0 0

File: save/5body.urdf (robot description, URDF)
Before this commit: robot robot, 4 links, 3 joints
Links:
- added link link4, mass 1; collision box size=0.8833676848800409 0.6485859189085685 0.6334813506332717; visual box size=0.8833676848800409 0.6485859189085685 0.6334813506332717
- added link link5, mass 1; collision box size=0.47270638215297983 0.2300868792772154 0.7843799267179494; visual box size=0.47270638215297983 0.2300868792772154 0.7843799267179494
- link link0: geometry collision box size=0.5187471549442595 0.33361851301769613 0.8708534894495175; visual box size=0.5187471549442595 0.33361851301769613 0.8708534894495175
- link link1: geometry collision box size=0.776927206683842 0.6808264392220617 0.7874542703739524; visual box size=0.776927206683842 0.6808264392220617 0.7874542703739524
- link link2: geometry collision box size=0.4521200678493451 0.26902138299267825 0.4967973753729892; visual box size=0.4521200678493451 0.26902138299267825 0.4967973753729892
- link link3: geometry collision box size=0.7415618613910955 0.3936604504078181 0.30138966595816447; visual box size=0.7415618613910955 0.3936604504078181 0.30138966595816447
Joints:
- added joint link3_link4: type revolute, parent link3, child link4, origin xyz=0.37078093069554774 0.19683022520390905 0 rpy=0 0 0, axis 1 0 1, limit lower=-3.14159 upper=3.14159 effort=0.0 velocity=0.0
- added joint link4_link5: type revolute, parent link4, child link5, origin xyz=0.8833676848800409 0 0 rpy=0 0 0, axis 1 0 1, limit lower=-3.14159 upper=3.14159 effort=0.0 velocity=0.0
- joint link0_link1: axis 1 0 0 -> 1 0 1; origin xyz=0.25 0 5 rpy=0 0 0 -> xyz=0 0 5.25937357747213 rpy=0 0 0
- joint link1_link2: axis 1 0 0 -> 1 0 1; origin xyz=0.4725097544487099 0 0.312111476573709 rpy=0 0 0 -> xyz=0 0.3404132196110308 0.3937271351869762 rpy=0 0 0
- joint link2_link3: axis 1 0 0 -> 1 0 1; origin xyz=0 0 0.6813510800855497 rpy=0 0 0 -> xyz=0 0.26902138299267825 0 rpy=0 0 0

File: save/6body.urdf (robot description, URDF)
Before this commit: robot robot, 4 links, 3 joints
Links:
- added link link4, mass 1; collision box size=0.6489590501069336 0.6395681576264207 0.5902552938561811; visual box size=0.6489590501069336 0.6395681576264207 0.5902552938561811
- added link link5, mass 1; collision box size=0.6761738731090681 0.32708676630508415 0.7924309631524438; visual box size=0.6761738731090681 0.32708676630508415 0.7924309631524438
- link link0: geometry collision box size=0.5187471549442595 0.33361851301769613 0.8708534894495175; visual box size=0.5187471549442595 0.33361851301769613 0.8708534894495175
- link link1: geometry collision box size=0.26696495182476065 0.7266575079261359 0.3001034351549571; visual box size=0.26696495182476065 0.7266575079261359 0.3001034351549571
- link link2: geometry collision box size=0.7870992354676485 0.7449907857288489 0.9568992397890697; visual box size=0.7870992354676485 0.7449907857288489 0.9568992397890697
- link link3: geometry collision box size=0.5731519138675956 0.4238640259576923 0.44724464947436354; visual box size=0.5731519138675956 0.4238640259576923 0.44724464947436354
Joints:
- added joint link3_link4: type revolute, parent link3, child link4, origin xyz=0.2865759569337978 0 0.22362232473718177 rpy=0 0 0, axis 0 1 0, limit lower=-3.14159 upper=3.14159 effort=0.0 velocity=0.0
- added joint link4_link5: type revolute, parent link4, child link5, origin xyz=0.6489590501069336 0 0 rpy=0 0 0, axis 0 1 0, limit lower=-3.14159 upper=3.14159 effort=0.0 velocity=0.0
- joint link0_link1: axis 1 0 0 -> 0 1 0; origin xyz=0 0 5.25 rpy=0 0 0 -> xyz=0 0.16680925650884806 5 rpy=0 0 0
- joint link1_link2: axis 1 0 0 -> 0 1 0; origin xyz=0 0.30932161131298497 0.3077584952988014 rpy=0 0 0 -> xyz=0 0.7266575079261359 0 rpy=0 0 0
- joint link2_link3: axis 1 0 0 -> 0 1 0; origin xyz=0 0.8739037675347314 0 rpy=0 0 0 -> xyz=0 0.37249539286442446 0.47844961989453483 rpy=0 0 0

File: save/7body.urdf (robot description, URDF)
Before this commit: robot robot, 4 links, 3 joints
Links:
- added link link4, mass 1; collision box size=0.2690784599054789 0.46625800037363024 0.5252639158490235; visual box size=0.2690784599054789 0.46625800037363024 0.5252639158490235
- added link link5, mass 1; collision box size=0.6676435158635925 0.451284118375762 0.652612768799465; visual box size=0.6676435158635925 0.451284118375762 0.652612768799465
- link link0: geometry collision box size=0.5187471549442595 0.33361851301769613 0.8708534894495175; visual box size=0.5187471549442595 0.33361851301769613 0.8708534894495175
- link link1: geometry collision box size=0.2530932139378547 0.43360669721419837 0.4478073585915975; visual box size=0.2530932139378547 0.43360669721419837 0.4478073585915975
- link link2: geometry collision box size=0.6232108233133041 0.334872830434361 0.8083105477133912; visual box size=0.6232108233133041 0.334872830434361 0.8083105477133912
- link link3: geometry collision box size=0.8071663654193499 0.3563839570163186 0.7395080747033631; visual box size=0.8071663654193499 0.3563839570163186 0.7395080747033631
Joints:
- added joint link3_link4: type revolute, parent link3, child link4, origin xyz=0.8071663654193499 0 0 rpy=0 0 0, axis 1 1 0, limit lower=-3.14159 upper=3.14159 effort=0.0 velocity=0.0
- added joint link4_link5: type revolute, parent link4, child link5, origin xyz=0.2690784599054789 0 0 rpy=0 0 0, axis 1 1 0, limit lower=-3.14159 upper=3.14159 effort=0.0 velocity=0.0
- joint link0_link1: axis 0 0 1 -> 1 1 0; origin xyz=0 0.25 5 rpy=0 0 0 -> xyz=0 0 5.25937357747213 rpy=0 0 0
- joint link1_link2: axis 0 0 1 -> 1 1 0; origin xyz=0 0.1958011679374607 0.10392351945621484 rpy=0 0 0 -> xyz=0 0 0.4478073585915975 rpy=0 0 0
- joint link2_link3: axis 0 0 1 -> 1 1 0; origin xyz=0 0.257160175576849 0.19970749530421925 rpy=0 0 0 -> xyz=0.31160541165665206 0 0.4041552738566956 rpy=0 0 0

File: save/9body.urdf (robot description, URDF)
Before this commit: robot robot, 4 links, 3 joints
Links:
- added link link4, mass 1; collision box size=0.4077547623083875 0.7651468296229287 0.4549747946563944; visual box size=0.4077547623083875 0.7651468296229287 0.4549747946563944
- added link link5, mass 1; collision box size=0.40670665860777994 0.35641939266111833 0.4569001436676954; visual box size=0.40670665860777994 0.35641939266111833 0.4569001436676954
- link link0: geometry collision box size=0.5187471549442595 0.33361851301769613 0.8708534894495175; visual box size=0.5187471549442595 0.33361851301769613 0.8708534894495175
- link link1: geometry collision box size=0.3543133897533717 0.8239359919540201 0.7146802687023277; visual box size=0.3543133897533717 0.8239359919540201 0.7146802687023277
- link link2: geometry collision box size=0.6612657984493984 0.447320864598771 0.8495896202347575; visual box size=0.6612657984493984 0.447320864598771 0.8495896202347575
- link link3: geometry collision box size=0.5249830620569577 0.5668819234566724 0.459983299067084; visual box size=0.5249830620569577 0.5668819234566724 0.459983299067084
Joints:
- added joint link3_link4: type revolute, parent link3, child link4, origin xyz=0 0.2834409617283362 0.229991649533542 rpy=0 0 0, axis 1 1 1, limit lower=-3.14159 upper=3.14159 effort=0.0 velocity=0.0
- added joint link4_link5: type revolute, parent link4, child link5, origin xyz=0.20387738115419374 0.38257341481146434 0 rpy=0 0 0, axis 1 1 1, limit lower=-3.14159 upper=3.14159 effort=0.0 velocity=0.0
- joint link0_link1: axis 0 0 1 -> 1 1 1; origin xyz=0 0 5.25 rpy=0 0 0 -> xyz=0.25937357747212975 0 5 rpy=0 0 0
- joint link1_link2: axis 0 0 1 -> 1 1 1; origin xyz=0 0.15513726991905932 0.38220928840823265 rpy=0 0 0 -> xyz=0.17715669487668584 0 0.35734013435116385 rpy=0 0 0
- joint link2_link3: axis 0 0 1 -> 1 1 1; origin xyz=0.4263732830654626 0.2366536230757033 0 rpy=0 0 0 -> xyz=0 0 0.8495896202347575 rpy=0 0 0
